File: POI/PovPOI/PovPOI.kicad_pcb (KiCad board)
At the start: 2 copper layers, 21.7 x 46 mm, 19 parts, among them J1 Conn_02x08_Top_Bottom, J2 Conn_02x08_Top_Bottom, J3 Conn_01x04, J5 Conn_01x04

Commit message: POV POI v2, working towards v3
Parts:
- removed BatteryOnSW1: SW_SPST, Connector_PinSocket_2.54mm:PinSocket_1x02_P2.54mm_Vertical
- removed C1: C_Polarized, Capacitor_THT:CP_Radial_D5.0mm_P2.50mm
- removed R1, R2: R_Small, Resistor_SMD:R_0805_2012Metric_Pad1.20x1.40mm_HandSolder
- added H4: MountingHole, MountingHole:MountingHole_2.2mm_M2, F.Cu at (45.7, 69.8)
- added H5: MountingHole, MountingHole:MountingHole_2.2mm_M2, F.Cu at (40.0, 38.1)
- added SW1: SW_SPDT, Connector_PinSocket_2.54mm:PinSocket_1x03_P2.54mm_Vertical, F.Cu at (38.1, 27.9)
- J3, J5: footprint Connector_PinHeader_2.54mm:PinHeader_1x04_P2.54mm_Horizontal -> Library:PinHeader_1x04_P2.54mm_Horizontal_Seth
- moved H1 27.9 mm to (45.7, 53.3)
- moved H3 27.0 mm to (27.9, 69.8)
- moved JP1 11.0 mm to (38.7, 30.5), turned to 0 degrees
- moved JP2 8.36 mm to (38.8, 33.0), turned to 0 degrees
- moved TP3 8.03 mm to (35.6, 35.6)
- moved H2 3.81 mm to (27.9, 53.3)
- moved TP4 3.59 mm to (35.6, 38.1)
- moved BatteryConn1 2.62 mm to (35.6, 53.3)
- moved TP1 2.54 mm to (35.6, 30.5)
- moved TP2 2.54 mm to (35.6, 33.0)
- moved C2 1.32 mm to (34.3, 50.2)
Connections:
- C2 pad 1: /PCB_BAT -> /BAT_TERMINAL
- J3 pad 2: /22 -> /19
- J3 pad 3: /23 -> /20
- J3 pad 4: /PCB_BAT -> /PCB_BAT_ON
- J5 pad 2: /22 -> /19
- J5 pad 3: /23 -> /20
- J5 pad 4: /PCB_BAT -> /PCB_BAT_ON
- JP1 pad 1: /PCB_BAT -> /PCB_BAT_ON
- JP2 pad 1: /PCB_BAT -> /PCB_BAT_ON
- TP1 pad 1: /CHIP_BAT+ -> /PCB_BAT_ON
Routing:
- net /PCB_BAT_ON: track 0.00 -> 58.2 mm
- net /PCB_BAT: track 48.4 -> 0.00 mm
- net GND: track 50.7 -> 3.29 mm
- net /23: track 42.4 -> 2.54 mm, vias 1 -> 0
- net /20: track 2.54 -> 34.7 mm
- net /19: track 2.54 -> 31.6 mm
- net /22: track 30.6 -> 2.54 mm
- net /BAT_TERMINAL: track 3.81 -> 27.9 mm
- net /CHIP_BAT+: track 20.4 -> 7.40 mm
- net /4: track 8.63 -> 2.54 mm
- net /VIN: track 18.7 -> 15.0 mm
- net /3V3: track 11.2 -> 8.67 mm
- added copper zone on F.Cu, net GND
Other:
- board size 21.7 x 46 mm -> 21.7 x 46.7 mm
- board text added: "19"
- board text added: "20"
- board text added: "3V3"
- board text added: "BAT+"
- board text added: "POV POI v2 Haus Anima 20240603 Zhigalka"
- board text added: "VIN"
- board text removed: "22"
- board text removed: "23"
- board text removed: "POV POI v1 Haus Anima 20240301 Zhigalka"

Commit message: POV POI v2.5 before accel import
Parts:
- removed JP1, JP2: SolderJumper_2_Open, Jumper:SolderJumper-2_P1.3mm_Open_RoundedPad1.0x1.5mm
- removed TP1, TP2, TP3, TP4: TestPoint, TestPoint:TestPoint_THTPad_D1.5mm_Drill0.7mm
- added C1: C_Polarized, Resistor_SMD:R_0805_2012Metric_Pad1.20x1.40mm_HandSolder, B.Cu at (38.4, 50.2)
- added R1: R_US, Resistor_SMD:R_0805_2012Metric_Pad1.20x1.40mm_HandSolder, B.Cu at (36.5, 31.1)
- added R2: R_US, Resistor_SMD:R_0805_2012Metric_Pad1.20x1.40mm_HandSolder, B.Cu at (36.5, 33.7)
- added U1: MC3479, Library:PQFN50P200X200X100-12N_HandSoldering, F.Cu at (37.1, 46.5)
- moved H5 24.9 mm to (64.8, 40.6)
- moved SW1 5.08 mm to (33.0, 27.9), turned to 90 degrees
- moved H3 2.84 mm to (29.2, 67.3)
- moved H4 2.84 mm to (44.5, 67.3)
- moved BatteryConn1 2.54 mm to (38.1, 53.3)
- moved H2 1.42 mm to (29.2, 52.7)
- moved H1 1.42 mm to (44.5, 52.7)
Connections:
- net /21 renamed /IO21
- net /22 renamed /IO22
- net /4 renamed /IO4
- J3 pad 4: /PCB_BAT_ON -> /CHIP_BAT+
- J5 pad 4: /PCB_BAT_ON -> /CHIP_BAT+
- SW1 pad 1: /PCB_BAT_ON -> /BAT_TERMINAL
- SW1 pad 3: /BAT_TERMINAL -> /CHIP_BAT+
Routing:
- net /PCB_BAT_ON: track 58.2 -> 0.00 mm
- net /CHIP_BAT+: track 7.40 -> 62.7 mm
- net /3V3: track 8.67 -> 35.7 mm, vias 0 -> 2
- net /IO4: track 2.54 -> 18.5 mm, vias 0 -> 1
- net /IO22: track 2.54 -> 15.7 mm, vias 0 -> 2
- net /IO21: track 2.54 -> 11.2 mm
- net /VIN: track 15.0 -> 9.04 mm, vias 0 -> 1
- net GND: track 3.29 -> 6.13 mm, vias 0 -> 1
- net /BAT_TERMINAL: track 27.9 -> 30.5 mm
- net /19: track 31.6 -> 30.6 mm
- added copper zone on B.Cu, net GND
Other:
- board text added: "BOT"
- board text added: "TOP"
- board text removed: "J1"

Commit message: Unknown changes in PovPOI
Parts:
- added SW2: SW_SPST, Button_Switch_THT:SW_Tactile_SPST_Angled_PTS645Vx39-2LFS, F.Cu at (31.1, 29.3)
- H1, H2, H3, H4, H5: footprint MountingHole:MountingHole_2.2mm_M2 -> MountingHole:MountingHole_2.2mm_M2_Pad
- SW1: footprint Connector_PinSocket_2.54mm:PinSocket_1x03_P2.54mm_Vertical -> Button_Switch_THT:SW_Slide_SPDT_Angled_CK_OS102011MA1Q; moved to B.Cu
- moved R1 8.46 mm to (35.3, 39.5)
- moved SW1 4.25 mm to (37.3, 27.9), turned to 0 degrees
- moved R2 3.27 mm to (35.3, 36.7)
Routing:
- net /IO4: track 18.5 -> 11.6 mm
- net /BAT_TERMINAL: track 30.5 -> 37.0 mm
- net /VIN: track 9.04 -> 15.1 mm
- net /CHIP_BAT+: track 62.7 -> 57.6 mm
- net GND: track 6.13 -> 2.54 mm
- net /3V3: track 35.7 -> 37.9 mm
- net /IO22: track 15.7 -> 14.9 mm
