File: POI/PovPOI/PovPOI.kicad_sch (KiCad schematic)
At the start: 19 parts, among them J1 Conn_02x08_Top_Bottom, J2 Conn_02x08_Top_Bottom, J3 Conn_01x04, J5 Conn_01x04

Commit message: POV POI v2, working towards v3
Parts:
- removed BatteryOnSW1: SW_SPST, Connector_PinSocket_2.54mm:PinSocket_1x02_P2.54mm_Vertical, symbol Switch:SW_SPST
- removed C1: C_Polarized, Capacitor_THT:CP_Radial_D5.0mm_P2.50mm, symbol Device:C_Polarized
- removed R1, R2: R_Small, Resistor_SMD:R_0805_2012Metric_Pad1.20x1.40mm_HandSolder, symbol Device:R_Small
- added H4, H5: MountingHole, MountingHole:MountingHole_2.2mm_M2, symbol Mechanical:MountingHole
- added R1, R2: R_US, Resistor_SMD:R_0805_2012Metric_Pad1.20x1.40mm_HandSolder, symbol Device:R_US
- added SW1: SW_SPDT, Connector_PinSocket_2.54mm:PinSocket_1x03_P2.54mm_Vertical, symbol Switch:SW_SPDT
- J3, J5: footprint Connector_PinHeader_2.54mm:PinHeader_1x04_P2.54mm_Horizontal -> Library:PinHeader_1x04_P2.54mm_Horizontal_Seth
Connections:
- net 19: now also J3.2 (Pin_2), J5.2 (Pin_2)
- net 20: now also J3.3 (Pin_3), J5.3 (Pin_3)
- net 22: no longer J3.2 (Pin_2), J5.2 (Pin_2)
- net 23: no longer J3.3 (Pin_3), J5.3 (Pin_3)
- net BAT_TERMINAL: now also C2.1, SW1.2 (B), SW1.3 (C)
- net CHIP_BAT+: no longer TP1.1
- net GND: now also R2.1
- net VIN: now also R1.2
- net 4 renamed IO4
- net IO4: now also R1.1, R2.2
- net PCB_BAT renamed PCB_BAT_ON
- net PCB_BAT_ON: now also TP1.1, SW1.1 (A); no longer C2.1
Other:
- note added: "According to DF Robot Spec GPIO0 -> ADC_CH2 connected to CHIP_BAT+ in a 1:1 voltage divider"
- note added: "Plans for V2 - Disconnect PCB_BAT+ not GND? - 3 pin switch at the top Used PCB_BAT <-> CHIP_BAT+ which worked great for running & charging"
- note removed: "Analog pin to measure battery voltage"

Commit message: POV POI v2.5 before accel import
Parts:
- removed JP1: SolderJumper_2_Open, Jumper:SolderJumper-2_P1.3mm_Open_RoundedPad1.0x1.5mm, symbol Jumper:SolderJumper_2_Bridged
- removed JP2: SolderJumper_2_Open, Jumper:SolderJumper-2_P1.3mm_Open_RoundedPad1.0x1.5mm, symbol Jumper:SolderJumper_2_Open
- removed TP1, TP2, TP3, TP4: TestPoint, TestPoint:TestPoint_THTPad_D1.5mm_Drill0.7mm, symbol Connector:TestPoint
- added C1: C_Polarized, Resistor_SMD:R_0805_2012Metric_Pad1.20x1.40mm_HandSolder, symbol Device:C_Polarized
- added U1: MC3479, Library:PQFN50P200X200X100-12N_HandSoldering, symbol MC3479:MC3479
Connections:
- net 3V3: now also C1.1, U1.2 (~{CS}), U1.9 (VDD)
- net BAT_TERMINAL: now also SW1.1 (A); no longer SW1.3 (C)
- net CHIP_BAT+: now also J3.4 (Pin_4), J5.4 (Pin_4), SW1.3 (C)
- net GND: now also C1.2, U1.3 (DOUT_A6), U1.6 (GND), U1.7 (VPP)
- net 21 renamed IO21
- net IO21: now also U1.4 (DIN_SDA)
- net 22 renamed IO22
- net IO22: now also U1.1 (SCK_SCL)
- removed net PCB_BAT_ON: J3.4 (Pin_4), J5.4 (Pin_4), SW1.1 (A)
Other:
- note added: "I2C uses SCL/SDA on Ports 22/21"
- note added: "Notes from V2 -> V3 - Removed BAT / CHIP_BAT+ solder jumper - Removed test points (2nd row has same points)"
- note added: "Plans for V3 - Footprint on bottom for switch - Footprint for button next to switch Future - Either I2c or SMT for accelerometer - Run Cap Sensor wires towards top (can just use the inside pin row) - Measure amp draw @ 4v for 36 WS2812s (obvs black)"
- note added: "measures V_USB to check for active charging"
- note added: "same same"
- note removed: "Fail safe to try and power from VIN instead of BAT+"
- note removed: "Plans for V2 - Disconnect PCB_BAT+ not GND? - 3 pin switch at the top Used PCB_BAT <-> CHIP_BAT+ which worked great for running & charging"
- moved on the sheet: SW1

Commit message: Unknown changes in PovPOI
Parts:
- added SW2: SW_SPST, Button_Switch_THT:SW_Tactile_SPST_Angled_PTS645Vx39-2LFS, symbol Switch:SW_SPST
- H1, H2, H3, H4, H5: footprint MountingHole:MountingHole_2.2mm_M2 -> MountingHole:MountingHole_2.2mm_M2_Pad
- SW1: footprint Connector_PinSocket_2.54mm:PinSocket_1x03_P2.54mm_Vertical -> Button_Switch_THT:SW_Slide_SPDT_Angled_CK_OS102011MA1Q
Connections:
- net 17: now also SW2.2 (B)
- net 3V3: now also SW2.1 (A)
Other:
- note added: "Plans for V3 - Footprint on bottom for switch - Footprint for button next to switch - Either I2c or SMT for accelerometer - Top Side & Bottom Side labels - Better Mount Holes Plans for V4 - Run Cap Sensor wires towards top"
- note removed: "Plans for V3 - Footprint on bottom for switch - Footprint for button next to switch Future - Either I2c or SMT for accelerometer - Run Cap Sensor wires towards top (can just use the inside pin row) - Measure amp draw @ 4v for 36 WS2812s (obvs black)"
Changed lines of the file:
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@@
+	(wire
+		(pts
+			(xy 72.39 50.8) (xy 76.2 50.8)
+		)
+		(stroke
+			(width 0)
+			(type default)
+		)
+	)
 	(wire
 		(pts
@@
 		(pts
 			(xy 54.61 85.09) (xy 67.31 85.09)
+		)
+		(stroke
+			(width 0)
+			(type default)
+		)
+	)
+	(wire
+		(pts
+			(xy 57.15 50.8) (xy 62.23 50.8)
 		)
 		(stroke
@@
 		)
 	)
-	(text "Plans for V3\n- Footprint on bottom for switch\n- Footprint for button next to switch\n\nFuture\n- Either I2c or SMT for accelerometer\n- Run Cap Sensor wires towards top (can just use the inside pin row)\n- Measure amp draw @ 4v for 36  WS2812s (obvs black)"
+	(text "Plans for V3\n\n- Footprint on bottom for switch\n- Footprint for button next to switch\n- Either I2c or SMT for accelerometer\n- Top Side & Bottom Side labels\n- Better Mount Holes\n\nPlans for V4\n- Run Cap Sensor wires towards top\n"
 		(exclude_from_sim no)
 		(at 103.886 70.612 0)
@@
 		)
 	)
+	(label "3V3"
+		(at 57.15 50.8 180)
+		(fields_autoplaced yes)
+		(effects
+			(font
+				(size 1.27 1.27)
+			)
+			(justify right bottom)
+		)
+	)
 	(label "20"
 		(at 72.39 97.79 0)
@@
 	(label "V_USB"
 		(at 88.9 88.9 0)
+		(fields_autoplaced yes)
+		(effects
+			(font
+				(size 1.27 1.27)
+			)
+			(justify left bottom)
+		)
+	)
+	(label "17"
+		(at 76.2 50.8 0)
 		(fields_autoplaced yes)
 		(effects
@@
 			)
 		)
-		(property "Footprint" "Connector_PinSocket_2.54mm:PinSocket_1x03_P2.54mm_Vertical"
+		(property "Footprint" "Button_Switch_THT:SW_Slide_SPDT_Angled_CK_OS102011MA1Q"
 			(at 57.15 39.37 0)
 			(effects
@@
 			)
 		)
-		(property "Footprint" "MountingHole:MountingHole_2.2mm_M2"
+		(property "Footprint" "MountingHole:MountingHole_2.2mm_M2_Pad"
 			(at 165.1 69.85 0)
 			(effects
@@
 	)
 	(symbol
+		(lib_id "Switch:SW_SPST")
+		(at 67.31 50.8 0)
+		(unit 1)
+		(exclude_from_sim no)
+		(in_bom yes)
+		(on_board yes)
+		(dnp no)
+		(property "Reference" "SW2"
+			(at 67.818 46.99 0)
+			(effects
+				(font
+					(size 1.27 1.27)
+				)
+			)
+		)
+		(property "Value" "SW_SPST"
+			(at 67.31 46.99 0)
+			(effects
+				(font
+					(size 1.27 1.27)
+				)
+				(hide yes)
+			)
+		)
+		(property "Footprint" "Button_Switch_THT:SW_Tactile_SPST_Angled_PTS645Vx39-2LFS"
+			(at 67.31 50.8 0)
+			(effects
+				(font
+					(size 1.27 1.27)
+				)
+				(hide yes)
+			)
+		)
+		(property "Datasheet" "~"
+			(at 67.31 50.8 0)
+			(effects
+				(font
+					(size 1.27 1.27)
+				)
+			)
+		)
+		(property "Description" "Single Pole Single Throw (SPST) switch"
+			(at 67.31 50.8 0)
+			(effects
+				(font
+					(size 1.27 1.27)
+				)
+				(hide yes)
+			)
+		)
+		(pin "2"
+		)
+		(pin "1"
+		)
+		(instances
+			(project ""
+				(path "/9cbb567e-c8f8-42fb-9f8f-dc1b70b902c7"
+					(reference "SW2")
+					(unit 1)
+				)
+			)
+		)
+	)
+	(symbol
 		(lib_id "Device:R_US")
 		(at 107.95 46.99 180)
@@
 			)
 		)
-		(property "Footprint" "MountingHole:MountingHole_2.2mm_M2"
+		(property "Footprint" "MountingHole:MountingHole_2.2mm_M2_Pad"
 			(at 165.1 57.15 0)
 			(effects
@@
 			)
 		)
-		(property "Footprint" "MountingHole:MountingHole_2.2mm_M2"
+		(property "Footprint" "MountingHole:MountingHole_2.2mm_M2_Pad"
 			(at 165.1 64.77 0)
 			(effects
@@
 			)
 		)
-		(property "Footprint" "MountingHole:MountingHole_2.2mm_M2"
+		(property "Footprint" "MountingHole:MountingHole_2.2mm_M2_Pad"
 			(at 160.02 64.77 0)
 			(effects
@@
 			)
 		)
-		(property "Footprint" "MountingHole:MountingHole_2.2mm_M2"
+		(property "Footprint" "MountingHole:MountingHole_2.2mm_M2_Pad"
 			(at 160.02 69.85 0)
 			(effects
